File: hardware/ioboard/ioboard.kicad_sch (KiCad schematic)
At the start: 11 parts, among them J1 IN1, J2 IN2, J3 IN3, J4 INV_OUT, J5 OUT, J6 CLIP_OUT, J7 Conn_01x06, J8 Conn_01x06

Commit message: Update `ioboard`
Parts:
- removed J7, J8: Conn_01x06, Connector_PinSocket_2.54mm:PinSocket_1x06_P2.54mm_Vertical, symbol Connector_Generic:Conn_01x06
- added J7: Conn_Upper, Connector_PinSocket_2.54mm:PinSocket_2x05_P2.54mm_Vertical_SMD, symbol Connector_Generic:Conn_02x05_Counter_Clockwise
- added J8: Conn_Lower, Connector_PinSocket_2.54mm:PinSocket_2x05_P2.54mm_Vertical_SMD, symbol Connector_Generic:Conn_02x05_Counter_Clockwise
- J4: value INV_OUT -> OUT1
- J5: value OUT -> OUT2
- J6: value CLIP_OUT -> OUT3
- RV1: value 100k -> POT1
- RV2: value 100k -> POT2
- RV3: value 100k -> POT3
Connections:
- net GND: now also J7.1 (Pin_1), J8.1 (Pin_1); no longer J1.TN, J2.TN, J3.TN, RV1.1, RV2.1, RV3.1
- net IN1: now also J1.T, J7.9 (Pin_9); no longer RV1.2
- net IN2: now also J2.T, J7.5 (Pin_5); no longer RV2.2
- net IN3: now also J3.T, J7.3 (Pin_3); no longer RV3.2
- net POT1_P3: now reaches RV1.3
- net POT1_P3: now also J7.4 (Pin_4); no longer J1.T
- net POT2_P3: now reaches RV2.3
- net POT2_P3: now also J8.4 (Pin_4); no longer J2.T
- net POT3_P3: now reaches RV3.3
- net POT3_P3: now also J8.3 (Pin_3); no longer J3.T
- net CLIP_OUT renamed OUT3
- net OUT3: now also J8.2 (Pin_2)
- net INV_OUT renamed OUT1
- net OUT1: now also J8.10 (Pin_10)
- net OUT renamed OUT2
- net OUT2: now also J8.6 (Pin_6)
- new net IN1_NORMAL: J1.TN, J7.10 (Pin_10)
- new net IN2_NORMAL: J2.TN, J7.7 (Pin_7)
- new net IN3_NORMAL: J3.TN, J7.2 (Pin_2)
- new net POT1_P1: J7.8 (Pin_8), RV1.1
- new net POT1_P2: J7.6 (Pin_6), RV1.2
- new net POT2_P1: J8.8 (Pin_8), RV2.1
- new net POT2_P2: J8.9 (Pin_9), RV2.2
- new net POT3_P1: J8.7 (Pin_7), RV3.1
- new net POT3_P2: J8.5 (Pin_5), RV3.2
Other:
- moved on the sheet: J1, J2, J3, J4, J5, J6, RV1, RV2, RV3
