File: hardware/ioboard/ioboard.kicad_pcb (KiCad board)
At the start: 2 copper layers, 28 x 110 mm, 11 parts, among them J1 IN1, J2 IN2, J3 IN3, J4 INV_OUT, J5 OUT, J6 CLIP_OUT, J7 Conn_01x06, J8 Conn_01x06

Commit message: Update `ioboard`
Parts:
- J4: value INV_OUT -> OUT1
- J5: value OUT -> OUT2
- J6: value CLIP_OUT -> OUT3
- J7: value Conn_01x06 -> Conn_Upper; footprint Connector_PinSocket_2.54mm:PinSocket_1x06_P2.54mm_Vertical -> Connector_PinSocket_2.54mm:PinSocket_2x05_P2.54mm_Vertical_SMD
- J8: value Conn_01x06 -> Conn_Lower; footprint Connector_PinSocket_2.54mm:PinSocket_1x06_P2.54mm_Vertical -> Connector_PinSocket_2.54mm:PinSocket_2x05_P2.54mm_Vertical_SMD
- RV1: value 100k -> POT1
- RV2: value 100k -> POT2
- RV3: value 100k -> POT3
- moved J7 6.63 mm to (64.0, 69.0)
- moved J8 6.63 mm to (64.0, 134.0)
Connections:
- J1 pad T: Net-(J1-PadT) -> IN1
- J1 pad TN: GND -> IN1_NORMAL
- J2 pad T: Net-(J2-PadT) -> IN2
- J2 pad TN: GND -> IN2_NORMAL
- J3 pad T: Net-(J3-PadT) -> IN3
- J3 pad TN: GND -> IN3_NORMAL
- J4 pad T: INV_OUT -> OUT1
- J5 pad T: OUT -> OUT2
- J6 pad T: CLIP_OUT -> OUT3
- J7 pad 1: IN3 -> GND
- J7 pad 2: GND -> IN3_NORMAL
- J7 pad 3: IN2 -> IN3
- J7 pad 4: GND -> POT1_P3
- J7 pad 5: IN1 -> IN2
- J7 pad 6: GND -> POT1_P2
- J8 pad 1: CLIP_OUT -> GND
- J8 pad 2: GND -> OUT3
- J8 pad 3: OUT -> POT3_P3
- J8 pad 4: GND -> POT2_P3
- J8 pad 5: INV_OUT -> POT3_P2
- J8 pad 6: GND -> OUT2
- RV1 pad 1: GND -> POT1_P1
- RV1 pad 2: IN1 -> POT1_P2
- RV1 pad 3: Net-(J1-PadT) -> POT1_P3
- RV2 pad 1: GND -> POT2_P1
- RV2 pad 2: IN2 -> POT2_P2
- RV2 pad 3: Net-(J2-PadT) -> POT2_P3
- RV3 pad 1: GND -> POT3_P1
- RV3 pad 2: IN3 -> POT3_P2
- RV3 pad 3: Net-(J3-PadT) -> POT3_P3
Routing:
- net Net-(J3-PadT): track 77.2 -> 0.00 mm
- net Net-(J2-PadT): track 55.5 -> 0.00 mm
- net Net-(J1-PadT): track 45.2 -> 0.00 mm
- net IN3: track 59.9 -> 18.1 mm
- net POT2_P1: track 0.00 -> 37.1 mm
- net POT2_P3: track 0.00 -> 36.7 mm
- net CLIP_OUT: track 30.2 -> 0.00 mm
- net POT2_P2: track 0.00 -> 30.0 mm
- net INV_OUT: track 29.1 -> 0.00 mm
- net OUT: track 28.8 -> 0.00 mm
- net OUT2: track 0.00 -> 24.2 mm
- net OUT1: track 0.00 -> 24.1 mm
- net OUT3: track 0.00 -> 24.1 mm
- net IN2: track 39.4 -> 17.1 mm
- net IN1_NORMAL: track 0.00 -> 15.5 mm
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Other:
- board text removed: "CLIP_OUT"
- board text removed: "GND"
- board text removed: "IN1"
- board text removed: "IN2"
- board text removed: "IN3"
- board text removed: "INV_OUT"
- board text removed: "OUT"

Commit message: Add labels
Other:
- board text added: "GND"
- board text added: "IN1"
- board text added: "IN1N"
- board text added: "IN2N"
- board text added: "IN3"
- board text added: "IN3N"
- board text added: "OUT1"
- board text added: "OUT2"
- board text added: "OUT3"
- board text added: "P1P1"
- board text added: "P1P2"
- board text added: "P1P3"
- board text added: "P2P1"
- board text added: "P2P2"
- board text added: "P2P3"
- board text added: "P3P1"
- board text added: "P3P2"
- board text added: "P3P3"
Changed lines of the file:
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@@
 			(at 0 -7.85 90)
 			(layer "B.Fab")
+			(hide yes)
 			(effects
 				(font
@@
 		(layer "Edge.Cuts")
 	)
+	(gr_text "P3P3"
+		(at 67.18 129.25 90)
+		(layer "B.SilkS")
+		(effects
+			(font
+				(size 1 1)
+				(thickness 0.1)
+			)
+			(justify right bottom mirror)
+		)
+	)
+	(gr_text "GND"
+		(at 69.76 129.25 90)
+		(layer "B.SilkS")
+		(effects
+			(font
+				(size 1 1)
+				(thickness 0.1)
+			)
+			(justify right bottom mirror)
+		)
+	)
+	(gr_text "P2P1"
+		(at 61.97 139 90)
+		(layer "B.SilkS")
+		(effects
+			(font
+				(size 1 1)
+				(thickness 0.1)
+			)
+			(justify left bottom mirror)
+		)
+	)
+	(gr_text "P1P2"
+		(at 64.59 73.56 90)
+		(layer "B.SilkS")
+		(effects
+			(font
+				(size 1 1)
+				(thickness 0.1)
+			)
+			(justify left bottom mirror)
+		)
+	)
+	(gr_text "GND"
+		(at 69.65 64.5 90)
+		(layer "B.SilkS")
+		(effects
+			(font
+				(size 1 1)
+				(thickness 0.1)
+			)
+			(justify right bottom mirror)
+		)
+	)
+	(gr_text "P3P2"
+		(at 64.64 129.25 90)
+		(layer "B.SilkS")
+		(effects
+			(font
+				(size 1 1)
+				(thickness 0.1)
+			)
+			(justify right bottom mirror)
+		)
+	)
+	(gr_text "IN2N"
+		(at 62.05 64.5 90)
+		(layer "B.SilkS")
+		(effects
+			(font
+				(size 1 1)
+				(thickness 0.1)
+			)
+			(justify right bottom mirror)
+		)
+	)
+	(gr_text "P3P1"
+		(at 62.02 129.25 90)
+		(layer "B.SilkS")
+		(effects
+			(font
+				(size 1 1)
+				(thickness 0.1)
+			)
+			(justify right bottom mirror)
+		)
+	)
+	(gr_text "P1P3"
+		(at 67.09 73.57 90)
+		(layer "B.SilkS")
+		(effects
+			(font
+				(size 1 1)
+				(thickness 0.1)
+			)
+			(justify left bottom mirror)
+		)
+	)
+	(gr_text "IN1"
+		(at 59.51 64.5 90)
+		(layer "B.SilkS")
+		(effects
+			(font
+				(size 1 1)
+				(thickness 0.1)
+			)
+			(justify right bottom mirror)
+		)
+	)
+	(gr_text "P2P2"
+		(at 59.52 129.25 90)
+		(layer "B.SilkS")
+		(effects
+			(font
+				(size 1 1)
+				(thickness 0.1)
+			)
+			(justify right bottom mirror)
+		)
+	)
+	(gr_text "OUT2"
+		(at 64.52 139 90)
+		(layer "B.SilkS")
+		(effects
+			(font
+				(size 1 1)
+				(thickness 0.1)
+			)
+			(justify left bottom mirror)
+		)
+	)
+	(gr_text "IN1N"
+		(at 57.02 71.78 90)
+		(layer "B.SilkS")
+		(effects
+			(font
+				(size 1 1)
+				(thickness 0.1)
+			)
+			(justify left bottom mirror)
+		)
+	)
+	(gr_text "P2P3"
+		(at 67.14 139 90)
+		(layer "B.SilkS")
+		(effects
+			(font
+				(size 1 1)
+				(thickness 0.1)
+			)
+			(justify left bottom mirror)
+		)
+	)
+	(gr_text "OUT1"
+		(at 59.42 139 90)
+		(layer "B.SilkS")
+		(effects
+			(font
+				(size 1 1)
+				(thickness 0.1)
+			)
+			(justify left bottom mirror)
+		)
+	)
+	(gr_text "P1P1"
+		(at 62.08 73.56 90)
+		(layer "B.SilkS")
+		(effects
+			(font
+				(size 1 1)
+				(thickness 0.1)
+			)
+			(justify left bottom mirror)
+		)
+	)
+	(gr_text "IN3N"
+		(at 72.25 71.75 90)
+		(layer "B.SilkS")
+		(effects
+			(font
+				(size 1 1)
+				(thickness 0.1)
+			)
+			(justify left bottom mirror)
+		)
+	)
+	(gr_text "IN3"
+		(at 67.16 64.5 90)
+		(layer "B.SilkS")
+		(effects
+			(font
+				(size 1 1)
+				(thickness 0.1)
+			)
+			(justify right bottom mirror)
+		)
+	)
+	(gr_text "OUT3"
+		(at 69.59 139 90)
+		(layer "B.SilkS")
+		(effects
+			(font
+				(size 1 1)
+				(thickness 0.1)
+			)
+			(justify left bottom mirror)
+		)
+	)
 	(dimension
