File: hardware/mainboard/mainboard.kicad_pcb (KiCad board)
At the start: 4 copper layers, 28 x 110 mm, 47 parts, among them J1 Power Connector, J2 IN1, J3 IN2, J4 IN3, J5 INV OUT, J6 OUT, J7 CLIP OUT, U1 TL074

Commit message: Re-arrange things
Parts:
- moved R3 7.79 mm to (64.0, 79.8)
- moved R4 0.84 mm to (64.0, 92.8)
- moved R5 0.84 mm to (64.0, 113.1)
Routing:
- net Net-(U1A--): track 46.4 -> 38.5 mm, vias 4 -> 3
- net Net-(R3-Pad1): track 2.38 -> 10.2 mm
- net Net-(R4-Pad1): track 2.38 -> 3.23 mm
- net Net-(R5-Pad1): track 2.63 -> 3.47 mm
Changed lines of the file:
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@@
 	(footprint "Resistor_SMD:R_0805_2012Metric_Pad1.20x1.40mm_HandSolder"
 		(layer "B.Cu")
-		(at 64 72 -90)
+		(at 63.96 79.79 -90)
 		(descr "Resistor SMD 0805 (2012 Metric), square (rectangular) end terminal, IPC-7351 nominal with elongated pad for handsoldering. (Body size source: IPC-SM-782 page 72, https://www.pcb-3d.com/wordpress/wp-content/uploads/ipc-sm-782a_amendment_1_and_2.pdf), generated with kicad-footprint-generator")
 		(tags "resistor handsolder")
@@
 	(footprint "Resistor_SMD:R_0805_2012Metric_Pad1.20x1.40mm_HandSolder"
 		(layer "B.Cu")
-		(at 64 92 -90)
+		(at 63.98 92.84 -90)
 		(descr "Resistor SMD 0805 (2012 Metric), square (rectangular) end terminal, IPC-7351 nominal with elongated pad for handsoldering. (Body size source: IPC-SM-782 page 72, https://www.pcb-3d.com/wordpress/wp-content/uploads/ipc-sm-782a_amendment_1_and_2.pdf), generated with kicad-footprint-generator")
 		(tags "resistor handsolder")
@@
 	(footprint "Resistor_SMD:R_0805_2012Metric_Pad1.20x1.40mm_HandSolder"
 		(layer "B.Cu")
-		(at 64 112.25 -90)
+		(at 63.99 113.09 -90)
 		(descr "Resistor SMD 0805 (2012 Metric), square (rectangular) end terminal, IPC-7351 nominal with elongated pad for handsoldering. (Body size source: IPC-SM-782 page 72, https://www.pcb-3d.com/wordpress/wp-content/uploads/ipc-sm-782a_amendment_1_and_2.pdf), generated with kicad-footprint-generator")
 		(tags "resistor handsolder")
@@
 	)
 	(gr_text "100k"
-		(at 62.5 90.1 90)
+		(at 62.71 90.96 90)
 		(layer "B.SilkS")
 		(effects
@@
 	)
 	(gr_text "100k"
-		(at 62.6 70.1 90)
+		(at 62.73 78 90)
 		(layer "B.SilkS")
 		(effects
@@
 	)
 	(gr_text "100k"
-		(at 62.7 110.3 90)
+		(at 62.78 111.21 90)
 		(layer "B.SilkS")
 		(effects
@@
 	)
 	(via
-		(at 64 80.4)
-		(size 0.6)
-		(drill 0.3)
-		(layers "F.Cu" "B.Cu")
-		(free yes)
-		(net 1)
-	)
-	(via
 		(at 60.2 133.8)
 		(size 0.6)
@@
 	)
 	(via
+		(at 63.67 104.34)
+		(size 0.6)
+		(drill 0.3)
+		(layers "F.Cu" "B.Cu")
+		(free yes)
+		(net 1)
+	)
+	(via
 		(at 61.5 100.54)
 		(size 0.6)
@@
 	)
 	(segment
-		(start 64 68.62)
-		(end 64 71)
+		(start 64 78.75)
+		(end 63.96 78.79)
 		(width 0.2)
 		(layer "B.Cu")
@@
 	)
 	(segment
-		(start 64 93)
-		(end 64 101.435786)
-		(width 0.2)
-		(layer "F.Cu")
-		(net 20)
-	)
-	(segment
-		(start 63.707107 102.142893)
-		(end 61.5 104.35)
+		(start 64 68.62)
+		(end 64 78.75)
 		(width 0.2)
-		(layer "F.Cu")
-		(net 20)
+		(layer "B.Cu")
+		(net 19)
 	)
 	(segment
-		(start 65.201 75.451)
-		(end 65.201 91.799)
+		(start 62.701 112.396786)
+		(end 62.701 105.965214)
 		(width 0.2)
 		(layer "F.Cu")
@@
 	)
 	(segment
-		(start 62.993893 112.243893)
-		(end 64 113.25)
+		(start 63.98 114.09)
+		(end 62.993893 113.103893)
 		(width 0.2)
 		(layer "F.Cu")
@@
 	)
 	(segment
-		(start 64 74.25)
-		(end 65.201 75.451)
+		(start 63.98 93.84)
+		(end 63.98 101.455786)
 		(width 0.2)
 		(layer "F.Cu")
@@
 	)
 	(segment
-		(start 65.201 91.799)
-		(end 64 93)
+		(start 63.99 114.09)
+		(end 63.98 114.09)
 		(width 0.2)
 		(layer "F.Cu")
@@
 	)
 	(segment
-		(start 62.701 105.965214)
-		(end 62.701 111.536786)
+		(start 63.687107 102.162893)
+		(end 61.5 104.35)
 		(width 0.2)
 		(layer "F.Cu")
@@
 	)
 	(segment
-		(start 61.5 104.35)
-		(end 62.408107 105.258107)
+		(start 62.408107 105.258107)
+		(end 61.5 104.35)
 		(width 0.2)
 		(layer "F.Cu")
@@
 	)
 	(via
-		(at 64 113.25)
-		(size 0.6)
-		(drill 0.3)
-		(layers "F.Cu" "B.Cu")
-		(net 20)
-	)
-	(via
-		(at 64 93)
+		(at 63.98 93.84)
 		(size 0.6)
 		(drill 0.3)
@@
 	)
 	(via
-		(at 64 74.25)
+		(at 63.99 114.09)
 		(size 0.6)
 		(drill 0.3)
@@
 	)
 	(arc
-		(start 62.993893 112.243893)
-		(mid 62.77712 111.91947)
-		(end 62.701 111.536786)
+		(start 62.993893 113.103893)
+		(mid 62.77712 112.77947)
+		(end 62.701 112.396786)
 		(width 0.2)
 		(layer "F.Cu")
@@
 	)
 	(arc
-		(start 64 101.435786)
-		(mid 63.92388 101.818469)
-		(end 63.707107 102.142893)
+		(start 63.687107 102.162893)
+		(mid 63.90388 101.83847)
+		(end 63.98 101.455786)
 		(width 0.2)
 		(layer "F.Cu")
@@
 	)
 	(segment
-		(start 64 113.25)
+		(start 63.99 114.09)
+		(end 63.99 116.49)
+		(width 0.2)
+		(layer "B.Cu")
+		(net 20)
+	)
+	(segment
+		(start 62.799 82.365214)
+		(end 62.799 92.244786)
+		(width 0.2)
+		(layer "B.Cu")
+		(net 20)
+	)
+	(segment
+		(start 63.091893 92.951893)
+		(end 63.98 93.84)
+		(width 0.2)
+		(layer "B.Cu")
+		(net 20)
+	)
+	(segment
+		(start 63.99 116.49)
 		(end 64 116.5)
 		(width 0.2)
@@
 	)
 	(segment
-		(start 64 73)
-		(end 64 74.25)
+		(start 63.96 80.79)
+		(end 63.091893 81.658107)
+		(width 0.2)
+		(layer "B.Cu")
+		(net 20)
+	)
+	(arc
+		(start 63.091893 92.951893)
+		(mid 62.87512 92.62747)
+		(end 62.799 92.244786)
+		(width 0.2)
+		(layer "B.Cu")
+		(net 20)
+	)
+	(arc
+		(start 62.799 82.365214)
+		(mid 62.87512 81.982531)
+		(end 63.091893 81.658107)
 		(width 0.2)
 		(layer "B.Cu")
@@
 	)
 	(segment
+		(start 64 91.82)
+		(end 63.98 91.84)
+		(width 0.2)
+		(layer "B.Cu")
+		(net 21)
+	)
+	(segment
 		(start 64 88.62)
-		(end 64 91)
+		(end 64 91.82)
 		(width 0.2)
 		(layer "B.Cu")
@@
 	)
 	(segment
+		(start 64 112.08)
+		(end 63.99 112.09)
+		(width 0.2)
+		(layer "B.Cu")
+		(net 22)
+	)
+	(segment
 		(start 64 108.62)
-		(end 64 111.25)
+		(end 64 112.08)
 		(width 0.2)
 		(layer "B.Cu")
@@
 	)
 	(segment
-		(start 51.8 125.1)
-		(end 59.735786 125.1)
+		(start 60.75 106.25)
+		(end 60.591893 106.408107)
 		(width 0.2)
 		(layer "F.Cu")
@@
 	)
 	(segment
-		(start 60.591893 110.691836)
-		(end 64 114.099943)
+		(start 51.8 125.1)
+		(end 59.735786 125.1)
 		(width 0.2)
 		(layer "F.Cu")
@@
 	)
 	(segment
-		(start 60.75 106.25)
-		(end 60.591893 106.408107)
+		(start 60.299 107.115214)
+		(end 60.299 112.914786)
 		(width 0.2)
 		(layer "F.Cu")
@@
 	)
 	(segment
-		(start 64 114.099943)
-		(end 64 118.5)
+		(start 60.442893 124.807107)
+		(end 64 121.25)
 		(width 0.2)
 		(layer "F.Cu")
@@
 	)
 	(segment
-		(start 60.442893 124.807107)
-		(end 64 121.25)
+		(start 64 117.444214)
+		(end 64 118.5)
 		(width 0.2)
 		(layer "F.Cu")
@@
 	)
 	(segment
-		(start 60.299 107.115214)
-		(end 60.299 109.984729)
+		(start 60.591893 113.621893)
+		(end 63.707107 116.737107)
 		(width 0.2)
 		(layer "F.Cu")
@@
 	)
 	(arc
-		(start 60.591893 106.408107)
-		(mid 60.37512 106.73253)
-		(end 60.299 107.115214)
+		(start 60.299 107.115214)
+		(mid 60.37512 106.732531)
+		(end 60.591893 106.408107)
+		(width 0.2)
+		(layer "F.Cu")
+		(net 23)
+	)
+	(arc
+		(start 64 117.444214)
+		(mid 63.92388 117.061531)
+		(end 63.707107 116.737107)
 		(width 0.2)
 		(layer "F.Cu")
@@
 	)
 	(arc
-		(start 60.591893 110.691836)
-		(mid 60.37512 110.367413)
-		(end 60.299 109.984729)
+		(start 60.299 112.914786)
+		(mid 60.37512 113.297469)
+		(end 60.591893 113.621893)
 		(width 0.2)
 		(layer "F.Cu")

Commit message: Update `mainboard`
Routing:
- removed copper zone on In1.Cu, net GND
- removed copper zone on In2.Cu, net GND
Other:
- copper layers 4 -> 2
Changed lines of the file:
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@@
 	(layers
 		(0 "F.Cu" signal)
-		(4 "In1.Cu" signal)
-		(6 "In2.Cu" signal)
 		(2 "B.Cu" signal)
 		(9 "F.Adhes" user "F.Adhesive")
@@
 			)
 			(layer "dielectric 1"
-				(type "prepreg")
-				(thickness 0.1)
-				(material "FR4")
-				(epsilon_r 4.5)
-				(loss_tangent 0.02)
-			)
-			(layer "In1.Cu"
-				(type "copper")
-				(thickness 0.035)
-			)
-			(layer "dielectric 2"
 				(type "core")
-				(thickness 1.24)
-				(material "FR4")
-				(epsilon_r 4.5)
-				(loss_tangent 0.02)
-			)
-			(layer "In2.Cu"
-				(type "copper")
-				(thickness 0.035)
-			)
-			(layer "dielectric 3"
-				(type "prepreg")
-				(thickness 0.1)
+				(thickness 1.51)
 				(material "FR4")
 				(epsilon_r 4.5)
@@
 			)
 		)
-	)
-	(zone
-		(net 1)
-		(net_name "GND")
-		(layer "In1.Cu")
-		(hatch edge 0.5)
-		(connect_pads
-			(clearance 0.5)
-		)
-		(min_thickness 0.25)
-		(filled_areas_thickness no)
-		(fill yes
-			(thermal_gap 0.5)
-			(thermal_bridge_width 0.5)
-		)
-		(polygon
-			(pts
-				(xy 78.5 49.5) (xy 49.5 49.5) (xy 49.5 160.5) (xy 78.5 160.5)
-			)
-		)
-	)
-	(zone
-		(net 1)
-		(net_name "GND")
-		(layer "In2.Cu")
-		(hatch edge 0.5)
-		(priority 1)
-		(connect_pads
-			(clearance 0.5)
-		)
-		(min_thickness 0.25)
-		(filled_areas_thickness no)
-		(fill yes
-			(thermal_gap 0.5)
-			(thermal_bridge_width 0.5)
-		)
-		(polygon
-			(pts
-				(xy 78.5 49.5) (xy 49.5 49.5) (xy 49.5 160.5) (xy 78.5 160.5)
-			)
-		)
